File: PCB/Pen_Plotter_RPI_Hat_V2/Power_Supply.kicad_sch (KiCad schematic)
At the start: 5 parts, among them J1 BARREL_JACK_12V, U2 BIDIRECTIONAL_LEVEL_SHIFTER_7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, U3 AP63357_BUCK_5V_REG_BREAKOUT_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

Commit message: Simplified design, began layout process
Parts:
- removed J1: BARREL_JACK_12V, symbol Connector:Barrel_Jack_Switch
- removed R?: 2k2, Pen_Plotter_Lib:THT_RESISTOR_WITH_VALUE, symbol Device:R
- removed R?: 10k, Pen_Plotter_Lib:THT_RESISTOR_WITH_VALUE, symbol Device:R
- removed U2: BIDIRECTIONAL_LEVEL_SHIFTER_757, Pen_Plotter_Lib:BIDIRECTIONAL_LEVEL_SHIFTER_575, symbol Pen_Plotter_Lib:BIDIRECTIONAL_LEVEL_SHIFTER_757
- removed U3: AP63357_BUCK_5V_REG_BREAKOUT_SMD, Pen_Plotter_Lib:AP63357_BUCK_5V_REG_BREAKOUT_SMD, symbol Pen_Plotter_Lib:AP63357_BUCK_5V_REG_BREAKOUT_SMD
Other:
- note removed: "5V_REGULATOR"
- note removed: "BARREL_JACK_12V"
- note removed: "LOGIC_LEVEL_SHIFTER"
